Commit message: Corrección de archivos URDF

File: URDF/Archivos_URDF/urdf/Archivos_URDF.urdf (robot description, URDF)
Before this commit: robot Solid_URDF, 7 links, 6 joints
Links:
- link Link_2: mass 0.029815 -> 0.0298150173902571; geometry collision mesh filename=package://Archivos_URDF/meshes/Link_2.STL; visual mesh filename=package://Archivos_URDF/meshes/Link_2.STL
- link Link_3: mass 0.10048 -> 0.100483555337623; geometry collision mesh filename=package://Archivos_URDF/meshes/Link_3.STL; visual mesh filename=package://Archivos_URDF/meshes/Link_3.STL
- link Link_4: mass 0.060766 -> 0.0607663214998903; geometry collision mesh filename=package://Archivos_URDF/meshes/Link_4.STL; visual mesh filename=package://Archivos_URDF/meshes/Link_4.STL
- link Link_5: mass 0.046012 -> 0.0460123556163477; geometry collision mesh filename=package://Archivos_URDF/meshes/Link_5.STL; visual mesh filename=package://Archivos_URDF/meshes/Link_5.STL
- link Link_6: mass 0.0082022 -> 0.00820216814692821; geometry collision mesh filename=package://Archivos_URDF/meshes/Link_6.STL; visual mesh filename=package://Archivos_URDF/meshes/Link_6.STL
- link Link_7: mass 0.0082022 -> 0.00820216814692821; geometry collision mesh filename=package://Archivos_URDF/meshes/Link_7.STL; visual mesh filename=package://Archivos_URDF/meshes/Link_7.STL
- link base_link: mass 0.51331 -> 0.513305048081214; geometry collision mesh filename=package://Archivos_URDF/meshes/base_link.STL; visual mesh filename=package://Archivos_URDF/meshes/base_link.STL
Joints:
- joint Joint_5: axis 0 0 1 -> 0 0 -1; origin xyz=-0.1483 -0.0125 0 rpy=3.1416 -1.5708 0 -> xyz=-0.1483 -0.0125 0 rpy=0 1.5708 0
- joint Joint_6: origin xyz=0 0.0025 0.038 rpy=0 0 0 -> xyz=0 0.0025 -0.038 rpy=-3.1416 0 3.1416
- joint Joint_7: origin xyz=0 0.0025 0.038 rpy=0 0 0 -> xyz=0 0.0025 -0.038 rpy=-3.1416 0 3.1416
